File: Hardware/KiCad Source Files/V3 Connector + IRLED.kicad_pcb (KiCad board)
At the start: 2 copper layers, 60 x 126.6 mm, 151 parts, among them J1 YK3210203000G, J2 USB4085-GF-A, J3 Conn_01x08, J4 YK3210203000G, J5 USB4085-GF-A, J6 USB1125-GF-B, Q1 IRLU024NPBF, Q2 IRLU024NPBF, Q3 Q_NMOS, U1 MC33063AP, U4 LM4040LP-2.0, U5 MCP4801, U6 MCP3202

Commit message: Finalized V3 Connector BOM based on testing on hardware.
Parts:
- R17: value 200R -> 1K
- R6: value 120R -> 1K
Changed lines of the file:
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@@
 			)
 		)
-		(property "Value" "200R"
+		(property "Value" "1K"
 			(at 3.81 2.37 0)
 			(layer "F.Fab")
@@
 			)
 		)
-		(property "Part Number" "MFR-25FRF52-200R"
+		(property "Part Number" "MFR-25FRF52-1K"
 			(at 0 0 0)
 			(unlocked yes)
@@
 			)
 		)
-		(property "Value" "120R"
+		(property "Value" "1K"
 			(at 3.81 2.37 90)
 			(layer "F.Fab")
@@
 			)
 		)
-		(property "Part Number" "MFR-25FTE52-120R"
+		(property "Part Number" "MFR-25FRF52-1K"
 			(at 0 0 90)
 			(unlocked yes)
@@
 		(sheetname "/CC Sink/")
 		(sheetfile "Strobe Generation.kicad_sch")
-		(attr through_hole dnp)
+		(attr through_hole)
 		(fp_line
 			(start 7.08 -1.37)
@@
 		(sheetname "/CC Sink/")
 		(sheetfile "Strobe Generation.kicad_sch")
-		(attr through_hole)
+		(attr through_hole dnp)
 		(fp_line
 			(start 7.08 1.37)
@@
 		(sheetname "/CC Sink/")
 		(sheetfile "Strobe Generation.kicad_sch")
-		(attr through_hole)
+		(attr through_hole dnp)
 		(fp_line
 			(start 6.580001 0)
